File: Hardware/Schematic/ESP32.sch (KiCad schematic (older format))
At the start: 9 parts

Commit message: Add files via upload
Parts:
- removed C? (x3): 0.1uF, symbol Device:C
- removed C?: 1.5pF, symbol Device:C
- removed C?: 1.2pF, symbol Device:C
- removed C?: 0.1uf, symbol Device:C
- removed IC?: ESP32-PICO-V3, ASSETS:ESP32PICOV3, symbol Regular_Use:ESP32-PICO-V3
- removed L?: L, symbol Device:L
- removed L?: 1.8nH, symbol Device:L
- added C? (x5): 0.1uF, symbol Device:C
- added C?: 1uF, symbol Device:C
- added C?: 10uF, symbol Device:C
- added C?: 2.4pF, symbol Device:C
- added C?: 3.9pF, symbol Device:C
- added C? (x2): 20pF, symbol Device:C
- added IC?: ESP32-C3, ASSETS:QFN50P500X500X90-33N-D, symbol Regular_Use:ESP32-C3
- added J?: SMA_Angled, ASSETS:SMA_angled, symbol Regular_Use:SMA_Angled
- added L?: 2nH, symbol Device:L
- added L?: 2.7nH, symbol Device:L
- added R? (x7): 0, symbol Device:R
- added R?: 10K, symbol Device:R
- added U?: W25Q32JVSS, Package_SO:SOIC-8_5.23x5.23mm_P1.27mm, symbol Memory_Flash:W25Q32JVSS
- added Y?: NX2012SA-32.768K-STD-MUB-1, ASSETS:NX2012SA32768KSTDMUB1, symbol Regular_Use:NX2012SA-32.768K-STD-MUB-1
- added Y?: NX2016SA-40M-STD-CZS-3, ASSETS:NX2016SA40MSTDCZS3, symbol Regular_Use:NX2016SA-40M-STD-CZS-3
Connections:
- net labels added: ESP_RX, EXP_TX, LNA, MTCK, MTDI, MTDO, MTMS, SPICLK, SPICSO, SPID, SPIHD, SPIQ, SPIWP, XTAL_32_N, XTAL_32_P, XTAL_N, XTAL_P
- wire segments 36 -> 106
- no-connect marks 8 -> 7

Commit message: Add files via upload
Parts:
- C31, C32, C33, C34, C35, C36, C37, C38, C39, C40, C41: renamed from C?; footprint (none) -> Capacitor_SMD:C_0402_1005Metric
- L4, L5: renamed from L?; footprint (none) -> Inductor_SMD:L_0402_1005Metric
- R17, R18, R19, R20, R21, R22, R23, R24: renamed from R?; footprint (none) -> Resistor_SMD:R_0402_1005Metric
- gave numbers to parts that had none: 5
