File: Hardware/Schematic/IMU.sch (KiCad schematic (older format))
At the start: 17 parts

Commit message: Add files via upload
Connections:
- net SCL renamed SCL_ALT
- net SCL_ALT: no longer R?.2, U?.20 (COM0)
- net SDA renamed SDA_ALT
- net SDA_ALT: no longer R?.2, U?.19 (COM1)
- new net SCL_IMU: R?.2, U?.20 (COM0)
- new net SDA_IMU: R?.2, U?.19 (COM1)
Changed lines of the file:
@@
 $Descr A4 11693 8268
 encoding utf-8
-Sheet 3 4
-Title ""
-Date ""
-Rev ""
-Comp ""
+Sheet 3 5
+Title "ProRTK: All in one Real Time Kinematic device"
+Date "2021-05-12"
+Rev "1"
+Comp "Blackshield Engineering"
 Comment1 ""
 Comment2 ""
@@
 	2400 4450 3000 4450
 Text GLabel 900  4250 0    50   Input ~ 0
-SCL
+SCL_IMU
 Text GLabel 900  4350 0    50   Input ~ 0
-SDA
+SDA_IMU
 Wire Wire Line
 	900  4350 1200 4350
@@
 $EndComp
 Text GLabel 9800 3600 2    50   Input ~ 0
-SCL
+SCL_ALT
 Text GLabel 9800 3800 2    50   Input ~ 0
-SDA
+SDA_ALT
 Wire Wire Line
 	9100 3800 9500 3800

Commit message: Add files via upload
Parts:
- added R25: 10K, Resistor_SMD:R_0402_1005Metric, symbol Device:R
- C17, C18, C19, C20, C21, C22, C23, C24: renamed from C?; footprint (none) -> Capacitor_SMD:C_0402_1005Metric
- R10, R11, R12, R13, R14, R15: renamed from R?; footprint (none) -> Resistor_SMD:R_0402_1005Metric
- gave numbers to parts that had none: 3
Connections:
- net +3V3: now also R25.1; no longer U4.5 (SDO)
- new net: R25.2, U4.5 (SDO)
- no-connect marks 0 -> 2

Commit message: Add files via upload
Parts:
- removed U3: MC-146, Crystal:Crystal_SMD_SeikoEpson_MC146-4Pin_6.7x1.5mm, symbol Regular_Use:MC-146
- added Y5: NX2012SA-32.768K-STD-MUB-1, ASSETS:NX2012SA32768KSTDMUB1, symbol Regular_Use:NX2012SA-32.768K-STD-MUB-1
Connections:
- net VDD is gone; now on net +3V3: C17.1, C19.1, C20.1, U2.28 (VDDIO), U2.3 (VDD)
- net at C21.2, U2.26 (XOUT32): now also Y5.2 (CRYSTAL_2)
- net at C22.2, U2.27 (XIN32): now also Y5.1 (CRYSTAL_1)
Changed lines of the file:
@@
 $Descr A4 11693 8268
 encoding utf-8
-Sheet 3 5
+Sheet 5 5
 Title "ProRTK: All in one Real Time Kinematic device"
 Date "2021-05-12"
@@
 Wire Wire Line
 	3500 3350 3500 2400
-$Comp
-L power:VDD #PWR?
-U 1 1 60A5D15C
-P 3500 2300
-AR Path="/60A5D15C" Ref="#PWR?"  Part="1"
-AR Path="/60A47002/60A5D15C" Ref="#PWR044"  Part="1"
-F 0 "#PWR044" H 3500 2150 50  0001 C CNN
-F 1 "VDD" H 3515 2473 50  0000 C CNN
-F 2 "" H 3500 2300 50  0001 C CNN
-F 3 "" H 3500 2300 50  0001 C CNN
-	1    3500 2300
-	1    0    0    -1
-$EndComp
 Wire Wire Line
 	3700 3350 3700 2400
@@
 Wire Wire Line
 	2200 2750 2200 2850
-$Comp
-L Regular_Use:MC-146 U?
-U 1 1 60A5D1D7
-P 5450 3900
-AR Path="/60A5D1D7" Ref="U?"  Part="1"
-AR Path="/60A47002/60A5D1D7" Ref="U3"  Part="1"
-F 0 "U3" H 5500 3600 50  0000 C CNN
-F 1 "MC-146" H 5750 3600 50  0000 C CNN
-F 2 "Crystal:Crystal_SMD_SeikoEpson_MC146-4Pin_6.7x1.5mm" H 5450 4050 50  0001 C CNN
-F 3 "https://www.mouser.in/datasheet/2/137/MC_146_en-1649537.pdf" H 5450 4050 50  0001 C CNN
-	1    5450 3900
-	1    0    0    1
-$EndComp
 Wire Wire Line
 	4200 3700 4200 3550
@@
 Connection ~ 5100 3850
 Wire Wire Line
-	5100 3850 5350 3850
-Wire Wire Line
-	6000 3700 6450 3700
-Wire Wire Line
 	6450 3700 6450 3400
 Wire Wire Line
 	6450 3400 5800 3400
-Wire Wire Line
-	6000 3850 6450 3850
-Wire Wire Line
-	6450 3850 6450 4100
 Wire Wire Line
 	6450 4100 5800 4100
@@
 	6650 3700 6650 3800
 Connection ~ 6450 3700
-Wire Wire Line
-	6450 3850 6450 3700
-Connection ~ 6450 3850
 Wire Wire Line
 	900  4250 1500 4250
@@
 Wire Wire Line
 	9100 3400 9900 3400
+$Comp
+L power:+3.3V #PWR?
+U 1 1 60A8B28F
+P 3500 2300
+AR Path="/60A8B28F" Ref="#PWR?"  Part="1"
+AR Path="/60A47002/60A8B28F" Ref="#PWR0101"  Part="1"
+F 0 "#PWR0101" H 3500 2150 50  0001 C CNN
+F 1 "+3.3V" H 3400 2450 50  0000 L CNN
+F 2 "" H 3500 2300 50  0001 C CNN
+F 3 "" H 3500 2300 50  0001 C CNN
+	1    3500 2300
+	1    0    0    -1
+$EndComp
+$Comp
+L Regular_Use:NX2012SA-32.768K-STD-MUB-1 Y?
+U 1 1 60A9684C
+P 5400 3850
+AR Path="/60A10196/60A9684C" Ref="Y?"  Part="1"
+AR Path="/60A47002/60A9684C" Ref="Y5"  Part="1"
+F 0 "Y5" H 6109 3846 50  0000 L CNN
+F 1 "NX2012SA-32.768K-STD-MUB-1" H 6109 3755 50  0000 L CNN
+F 2 "ASSETS:NX2012SA32768KSTDMUB1" H 6450 3950 50  0001 L CNN
+F 3 "https://www.mouser.de/datasheet/2/905/c_NX2012SA-STD-MUB-1_e-1317508.pdf" H 6450 3850 50  0001 L CNN
+F 4 "NDK 32.76kHz Crystal Unit +/-20ppm SMD 2-Pin 2.05 x 1.2 x 0.55mm" H 6450 3750 50  0001 L CNN "Description"
+F 5 "0.6" H 6450 3650 50  0001 L CNN "Height"
+F 6 "344-NX2012SA32768K1" H 6450 3550 50  0001 L CNN "Mouser Part Number"
+F 7 "https://www.mouser.co.uk/ProductDetail/NDK/NX2012SA-32768K-STD-MUB-1?qs=55YtniHzbhA%252B6%2Fl1MwFZaQ%3D%3D" H 6450 3450 50  0001 L CNN "Mouser Price/Stock"
+F 8 "NDK" H 6450 3350 50  0001 L CNN "Manufacturer_Name"
+F 9 "NX2012SA-32.768K-STD-MUB-1" H 6450 3250 50  0001 L CNN "Manufacturer_Part_Number"
+	1    5400 3850
+	1    0    0    1
+$EndComp
+Wire Wire Line
+	6450 3700 6450 4100
+Wire Wire Line
+	5350 3700 5350 3750
+Wire Wire Line
+	5350 3750 5400 3750
+Wire Wire Line
+	5100 3850 5400 3850
 $EndSCHEMATC
