File: Hardware/Schematic/GNSS.sch (KiCad schematic (older format))
At the start: 1 part

Commit message: Add files via upload
Parts:
- added C? (x3): 56pF, symbol Device:C
- added C?: 1nF, symbol Device:C
- added C? (x2): 120pF, symbol Device:C
- added J?: SMA_Vertical, ASSETS:SMA_Vertical, symbol Regular_Use:SMA_Vertical
- added L?: 27nH, symbol Device:L
- added L?: 5nF, symbol Device:L
- added R?: 10K, symbol Device:R
- added U?: BGA725L6E6327FTSA1, ASSETS:BGA725L6E6327, symbol Regular_Use:BGA725L6E6327FTSA1
- added U?: B4327, ASSETS:B4327, symbol Regular_Use:B4327
Connections:
- net GND: now reaches U?.1 (GND)
- net GND: now also U?.10 (GND_RF), U?.12 (GND_RF), C?.2, C?.2, C?.2, C?.2, J?.2, J?.3 (2), J?.4 (2), J?.5 (2), R?.2, U?.1 (GND), U?.2 (GND), U?.3 (GND), U?.4 (GNDRF), U?.5 (GND)
- net at U?.11 (RF_IN): now also C?.2
- net at U?.13 (ANT_OFF): now also R?.1, U?.6 (PON)
- net VDD: now reaches U?.14 (VCC_RF)
- net VDD: now also C?.1, C?.1, U?.2 (VCC)
- net TX_GNSS: now reaches U?.2 (TX)
- net RX_GNSS: now reaches U?.3 (RX)
- net 1PPS: now reaches U?.4 (1PPS)
- net WAKE-UP: now reaches U?.5 (WAKE-UP)
- net VBAT: now reaches U?.6 (VBATT)
- net at U?.7 (VCC_IO): now also U?.8 (VCC), C?.1, L?.1
- net SYS_RSTN: now reaches U?.9 (SYS_RSTN)
- new net: C?.1, U?.4 (RF_IN)
- new net: C?.1, L?.1
- new net: L?.2, U?.5 (AI)
- new net: C?.2, J?.1
- new net: U?.1 (RF_OUT), U?.3 (AO)
- new net +3V3: C?.1, L?.2
Other:
- moved on the sheet: U?

Commit message: Add files via upload
Parts:
- removed J?: SMA_Vertical, ASSETS:SMA_Vertical, symbol Regular_Use:SMA_Vertical
- added J5: SMA_Angled, ASSETS:SMA_angled, symbol Regular_Use:SMA_Angled
- C25, C26, C27, C28, C29, C30: renamed from C?; footprint (none) -> Capacitor_SMD:C_0402_1005Metric
- L2, L3: renamed from L?; footprint (none) -> Inductor_SMD:L_0402_1005Metric
- R16: renamed from R?; footprint (none) -> Resistor_SMD:R_0402_1005Metric
- gave numbers to parts that had none: 3
Connections:
- net GND: now also J5.2, J5.3 (2), J5.4 (2), J5.5 (2)
- net at C25.2: now also J5.1
Changed lines of the file:
@@
 	1350 3800 1350 4100
 $Comp
-L power:GND #PWR?
+L power:GND #PWR062
 U 1 1 609E47A9
 P 1350 4100
-F 0 "#PWR?" H 1350 3850 50  0001 C CNN
+F 0 "#PWR062" H 1350 3850 50  0001 C CNN
 F 1 "GND" H 1350 3950 50  0000 C CNN
 F 2 "" H 1350 4100 50  0001 C CNN
@@
 Wire Wire Line
 	1350 3600 1450 3600
-$Comp
-L Regular_Use:SMA_Vertical J?
-U 1 1 609E26A1
-P 1250 3700
-F 0 "J?" H 1212 4014 50  0000 C CNN
-F 1 "SMA_Vertical" H 1212 3923 50  0000 C CNN
-F 2 "ASSETS:SMA_Vertical" H 1250 3700 50  0001 L BNN
-F 3 "https://www.te.com/usa-en/product-518148321.html?te_bu=Cor&te_type=disp&te_campaign=seda_glo_cor-seda-global-disp-prtnr-fy19-seda-model-bom-cta_sma-317_1&elqCampaignId=32493" H 1250 3700 50  0001 L BNN
-	1    1250 3700
-	1    0    0    -1
-$EndComp
 Wire Wire Line
 	2150 3600 2300 3600
@@
 	1750 3600 1850 3600
 $Comp
-L Device:C C?
+L Device:C C25
 U 1 1 609DFFF4
 P 1600 3600
-F 0 "C?" V 1348 3600 50  0000 C CNN
+F 0 "C25" V 1348 3600 50  0000 C CNN
 F 1 "120pF" V 1439 3600 50  0000 C CNN
-F 2 "" H 1638 3450 50  0001 C CNN
+F 2 "Capacitor_SMD:C_0402_1005Metric" H 1638 3450 50  0001 C CNN
 F 3 "~" H 1600 3600 50  0001 C CNN
 	1    1600 3600
@@
 $EndComp
 $Comp
-L Device:L L?
+L Device:L L2
 U 1 1 609DF956
 P 2000 3600
-F 0 "L?" V 2190 3600 50  0000 C CNN
+F 0 "L2" V 2190 3600 50  0000 C CNN
 F 1 "5nF" V 2099 3600 50  0000 C CNN
-F 2 "" H 2000 3600 50  0001 C CNN
+F 2 "Inductor_SMD:L_0402_1005Metric" H 2000 3600 50  0001 C CNN
 F 3 "~" H 2000 3600 50  0001 C CNN
 	1    2000 3600
@@
 $EndComp
 $Comp
-L power:GND #PWR?
+L power:GND #PWR067
 U 1 1 609D9935
 P 5800 3900
-F 0 "#PWR?" H 5800 3650 50  0001 C CNN
+F 0 "#PWR067" H 5800 3650 50  0001 C CNN
 F 1 "GND" H 5800 3750 50  0000 C CNN
 F 2 "" H 5800 3900 50  0001 C CNN
@@
 	5800 3550 5800 3000
 $Comp
-L Device:R R?
+L Device:R R16
 U 1 1 609D754D
 P 5800 3700
-F 0 "R?" H 5870 3746 50  0000 L CNN
+F 0 "R16" H 5870 3746 50  0000 L CNN
 F 1 "10K" H 5870 3655 50  0000 L CNN
-F 2 "" V 5730 3700 50  0001 C CNN
+F 2 "Resistor_SMD:R_0402_1005Metric" V 5730 3700 50  0001 C CNN
 F 3 "~" H 5800 3700 50  0001 C CNN
 	1    5800 3700
@@
 	5250 3450 5050 3450
 $Comp
-L Device:C C?
+L Device:C C27
 U 1 1 609D1FBB
 P 5400 3450
-F 0 "C?" V 5550 3400 50  0000 L CNN
+F 0 "C27" V 5550 3400 50  0000 L CNN
 F 1 "120pF" V 5250 3300 50  0000 L CNN
-F 2 "" H 5438 3300 50  0001 C CNN
+F 2 "Capacitor_SMD:C_0402_1005Metric" H 5438 3300 50  0001 C CNN
 F 3 "~" H 5400 3450 50  0001 C CNN
 	1    5400 3450
@@
 	4650 4100 4650 4050
 $Comp
-L power:GND #PWR?
+L power:GND #PWR066
 U 1 1 609CCCE1
 P 4650 4100
-F 0 "#PWR?" H 4650 3850 50  0001 C CNN
+F 0 "#PWR066" H 4650 3850 50  0001 C CNN
 F 1 "GND" H 4650 3950 50  0000 C CNN
 F 2 "" H 4650 4100 50  0001 C CNN
@@
 	3300 3900 3500 3900
 $Comp
-L power:GND #PWR?
+L power:GND #PWR064
 U 1 1 609CBAAF
 P 3500 4200
-F 0 "#PWR?" H 3500 3950 50  0001 C CNN
+F 0 "#PWR064" H 3500 3950 50  0001 C CNN
 F 1 "GND" H 3500 4050 50  0000 C CNN
 F 2 "" H 3500 4200 50  0001 C CNN
@@
 	3750 3050 3750 2950
 $Comp
-L power:GND #PWR?
+L power:GND #PWR065
 U 1 1 609C7E7B
 P 3750 3050
-F 0 "#PWR?" H 3750 2800 50  0001 C CNN
+F 0 "#PWR065" H 3750 2800 50  0001 C CNN
 F 1 "GND" H 3750 2900 50  0000 C CNN
 F 2 "" H 3750 3050 50  0001 C CNN
@@
 $EndComp
 $Comp
-L Device:C C?
+L Device:C C26
 U 1 1 609C7E75
 P 3750 2800
-F 0 "C?" H 3865 2846 50  0000 L CNN
+F 0 "C26" H 3865 2846 50  0000 L CNN
 F 1 "1nF" H 3865 2755 50  0000 L CNN
-F 2 "" H 3788 2650 50  0001 C CNN
+F 2 "Capacitor_SMD:C_0402_1005Metric" H 3788 2650 50  0001 C CNN
 F 3 "~" H 3750 2800 50  0001 C CNN
 	1    3750 2800
@@
 $EndComp
 $Comp
-L power:VDD #PWR?
+L power:VDD #PWR063
 U 1 1 609C5138
 P 3400 2350
-F 0 "#PWR?" H 3400 2200 50  0001 C CNN
+F 0 "#PWR063" H 3400 2200 50  0001 C CNN
 F 1 "VDD" H 3415 2523 50  0000 C CNN
 F 2 "" H 3400 2350 50  0001 C CNN
@@
 	4200 3450 3300 3450
 $Comp
-L Regular_Use:B4327 U?
+L Regular_Use:B4327 U6
 U 1 1 60A7E913
 P 4650 3450
-F 0 "U?" H 4625 3765 50  0000 C CNN
+F 0 "U6" H 4625 3765 50  0000 C CNN
 F 1 "B4327" H 4625 3674 50  0000 C CNN
 F 2 "ASSETS:B4327" H 4450 3650 50  0001 C CNN
@@
 	7100 3200 7050 3200
 $Comp
-L power:GND #PWR?
+L power:GND #PWR069
 U 1 1 60A7B9E9
 P 6600 3100
-F 0 "#PWR?" H 6600 2850 50  0001 C CNN
+F 0 "#PWR069" H 6600 2850 50  0001 C CNN
 F 1 "GND" H 6605 2927 50  0000 C CNN
 F 2 "" H 6600 3100 50  0001 C CNN
@@
 	7100 3750 6900 3750
 $Comp
-L Regular_Use:BGA725L6E6327FTSA1 U?
+L Regular_Use:BGA725L6E6327FTSA1 U5
 U 1 1 60A71222
 P 2800 3600
-F 0 "U?" H 2800 4167 50  0000 C CNN
+F 0 "U5" H 2800 4167 50  0000 C CNN
 F 1 "BGA725L6E6327FTSA1" H 2800 4076 50  0000 C CNN
 F 2 "ASSETS:BGA725L6E6327" H 2800 3600 50  0001 L BNN
@@
 $EndComp
 $Comp
-L power:VDD #PWR?
+L power:VDD #PWR068
 U 1 1 60A707E6
 P 6450 3750
-F 0 "#PWR?" H 6450 3600 50  0001 C CNN
+F 0 "#PWR068" H 6450 3600 50  0001 C CNN
 F 1 "VDD" H 6465 3923 50  0000 C CNN
 F 2 "" H 6450 3750 50  0001 C CNN
@@
 	10450 3950 10450 3850
 $Comp
-L power:GND #PWR?
+L power:GND #PWR073
 U 1 1 609B3EBA
 P 10450 3950
-F 0 "#PWR?" H 10450 3700 50  0001 C CNN
+F 0 "#PWR073" H 10450 3700 50  0001 C CNN
 F 1 "GND" H 10455 3777 50  0000 C CNN
 F 2 "" H 10450 3950 50  0001 C CNN
@@
 $EndComp
 $Comp
-L Device:C C?
+L Device:C C30
 U 1 1 609B3EB4
 P 10450 3700
-F 0 "C?" H 10565 3746 50  0000 L CNN
+F 0 "C30" H 10565 3746 50  0000 L CNN
 F 1 "56pF" H 10565 3655 50  0000 L CNN
-F 2 "" H 10488 3550 50  0001 C CNN
+F 2 "Capacitor_SMD:C_0402_1005Metric" H 10488 3550 50  0001 C CNN
 F 3 "~" H 10450 3700 50  0001 C CNN
 	1    10450 3700
@@
 $EndComp
 Wire Wire Line
-	9800 3400 8950 3400
+	9800 3400 9250 3400
 Connection ~ 9800 3400
 Wire Wire Line
@@
 	9800 3950 9800 3850
 $Comp
-L power:GND #PWR?
+L power:GND #PWR072
 U 1 1 609B35AC
 P 9800 3950
-F 0 "#PWR?" H 9800 3700 50  0001 C CNN
+F 0 "#PWR072" H 9800 3700 50  0001 C CNN
 F 1 "GND" H 9805 3777 50  0000 C CNN
 F 2 "" H 9800 3950 50  0001 C CNN
@@
 $EndComp
 $Comp
-L Device:C C?
+L Device:C C29
 U 1 1 609B35A6
 P 9800 3700
-F 0 "C?" H 9915 3746 50  0000 L CNN
+F 0 "C29" H 9915 3746 50  0000 L CNN
 F 1 "56pF" H 9915 3655 50  0000 L CNN
-F 2 "" H 9838 3550 50  0001 C CNN
+F 2 "Capacitor_SMD:C_0402_1005Metric" H 9838 3550 50  0001 C CNN
 F 3 "~" H 9800 3700 50  0001 C CNN
 	1    9800 3700
@@
 	7000 4050 6900 4050
 $Comp
-L power:GND #PWR?
+L power:GND #PWR070
 U 1 1 609B1DC2
 P 7000 4050
-F 0 "#PWR?" H 7000 3800 50  0001 C CNN
+F 0 "#PWR070" H 7000 3800 50  0001 C CNN
 F 1 "GND" V 7000 3850 50  0000 C CNN
 F 2 "" H 7000 4050 50  0001 C CNN
@@
 $EndComp
 $Comp
-L Device:C C?
+L Device:C C28
 U 1 1 609B1664
 P 6900 3900
-F 0 "C?" H 7015 3946 50  0000 L CNN
+F 0 "C28" H 7015 3946 50  0000 L CNN
 F 1 "56pF" H 7015 3855 50  0000 L CNN
-F 2 "" H 6938 3750 50  0001 C CNN
+F 2 "Capacitor_SMD:C_0402_1005Metric" H 6938 3750 50  0001 C CNN
 F 3 "~" H 6900 3900 50  0001 C CNN
 	1    6900 3900
@@
 	8500 3200 8650 3200
 $Comp
-L power:+3V3 #PWR?
+L power:+3V3 #PWR074
 U 1 1 609AF4F8
 P 10650 3250
-F 0 "#PWR?" H 10650 3100 50  0001 C CNN
+F 0 "#PWR074" H 10650 3100 50  0001 C CNN
 F 1 "+3V3" H 10665 3423 50  0000 C CNN
 F 2 "" H 10650 3250 50  0001 C CNN
@@
 	9950 3400 9800 3400
 $Comp
-L Device:L L?
+L Device:L L3
 U 1 1 609AEC35
 P 10100 3400
-F 0 "L?" V 10290 3400 50  0000 C CNN
+F 0 "L3" V 10290 3400 50  0000 C CNN
 F 1 "27nH" V 10199 3400 50  0000 C CNN
-F 2 "" H 10100 3400 50  0001 C CNN
+F 2 "Inductor_SMD:L_0402_1005Metric" H 10100 3400 50  0001 C CNN
 F 3 "~" H 10100 3400 50  0001 C CNN
 	1    10100 3400
@@
 P 7800 3900
 AR Path="/60BFDA09" Ref="U?"  Part="1"
-AR Path="/60BF870D/60BFDA09" Ref="U?"  Part="1"
-F 0 "U?" H 7800 4865 50  0000 C CNN
+AR Path="/60BF870D/60BFDA09" Ref="U7"  Part="1"
+F 0 "U7" H 7800 4865 50  0000 C CNN
 F 1 "TESEO-LIV3F" H 7800 4774 50  0000 C CNN
 F 2 "ASSETS:TESEO-LIV3F" H 7800 3900 50  0001 L BNN
@@
 	8600 4700 8600 4600
 $Comp
-L power:GND #PWR?
+L power:GND #PWR071
 U 1 1 609EF86D
 P 8600 4700
-F 0 "#PWR?" H 8600 4450 50  0001 C CNN
+F 0 "#PWR071" H 8600 4450 50  0001 C CNN
 F 1 "GND" H 8605 4527 50  0000 C CNN
 F 2 "" H 8600 4700 50  0001 C CNN
@@
 Text GLabel 9000 4200 2    50   Input ~ 0
 RX_GNSS
+$Comp
+L power:PWR_FLAG #FLG01
+U 1 1 60B4907C
+P 9250 3100
+F 0 "#FLG01" H 9250 3175 50  0001 C CNN
+F 1 "PWR_FLAG" H 9250 3273 50  0000 C CNN
+F 2 "" H 9250 3100 50  0001 C CNN
+F 3 "~" H 9250 3100 50  0001 C CNN
+	1    9250 3100
+	1    0    0    -1
+$EndComp
+Wire Wire Line
+	9250 3100 9250 3400
+Connection ~ 9250 3400
+Wire Wire Line
+	9250 3400 8950 3400
+$Comp
+L Regular_Use:SMA_Angled J5
+U 1 1 60BB13DA
+P 1250 3700
+F 0 "J5" H 1212 4014 50  0000 C CNN
+F 1 "SMA_Angled" H 1212 3923 50  0000 C CNN
+F 2 "ASSETS:SMA_angled" H 1250 3700 50  0001 L BNN
+F 3 "Compliant with Exemptions" H 1250 3700 50  0001 L BNN
+F 4 "https://www.te.com/usa-en/product-221790-1.html?te_bu=Cor&te_type=disp&te_campaign=seda_glo_cor-seda-global-disp-prtnr-fy19-seda-model-bom-cta_sma-317_1&elqCampaignId=32493" H 1250 3700 50  0001 L BNN "Field4"
+F 5 "221790-1" H 1250 3700 50  0001 L BNN "Field5"
+F 6 "1" H 1250 3700 50  0001 L BNN "Field6"
+	1    1250 3700
+	1    0    0    -1
+$EndComp
 $EndSCHEMATC

Commit message: Add files via upload
Parts:
- added U10, U11, U12, U9: RF_Taper, ASSETS:KL_Taper, symbol Regular_Use:RF_Taper
Connections:
- net at C27.1, U6.4 (RF_IN): now also U12.1 (Tap)
- net at L2.2, U5.5 (AI): now also U9.1 (Tap)
- net at U5.3 (AO), U6.1 (RF_OUT): now also U10.1 (Tap), U11.1 (Tap)
- no-connect marks 0 -> 1
Other:
- moved on the sheet: C26
Changed lines of the file:
@@
 $Descr A4 11693 8268
 encoding utf-8
-Sheet 4 5
+Sheet 3 5
 Title "ProRTK: All in one Real Time Kinematic device"
 Date "2021-05-12"
@@
 	1350 3600 1450 3600
 Wire Wire Line
-	2150 3600 2300 3600
+	2150 3600 2250 3600
 Wire Wire Line
 	1750 3600 1850 3600
@@
 	5550 3450 7100 3450
 Wire Wire Line
-	5250 3450 5050 3450
+	5250 3450 5150 3450
 $Comp
 L Device:C C27
@@
 	3300 3800 3500 3800
 Wire Wire Line
-	3400 2450 3400 2350
-Connection ~ 3400 2450
-Wire Wire Line
-	3750 2450 3400 2450
-Wire Wire Line
-	3750 2650 3750 2450
-Wire Wire Line
-	3750 3050 3750 2950
+	3400 2100 3400 2000
+Connection ~ 3400 2100
+Wire Wire Line
+	3050 2100 3400 2100
+Wire Wire Line
+	3050 2300 3050 2100
+Wire Wire Line
+	3050 2700 3050 2600
 $Comp
 L power:GND #PWR065
 U 1 1 609C7E7B
-P 3750 3050
-F 0 "#PWR065" H 3750 2800 50  0001 C CNN
-F 1 "GND" H 3750 2900 50  0000 C CNN
-F 2 "" H 3750 3050 50  0001 C CNN
-F 3 "" H 3750 3050 50  0001 C CNN
-	1    3750 3050
-	-1   0    0    -1
+P 3050 2700
+F 0 "#PWR065" H 3050 2450 50  0001 C CNN
+F 1 "GND" H 3050 2550 50  0000 C CNN
+F 2 "" H 3050 2700 50  0001 C CNN
+F 3 "" H 3050 2700 50  0001 C CNN
+	1    3050 2700
+	1    0    0    -1
 $EndComp
 $Comp
 L Device:C C26
 U 1 1 609C7E75
-P 3750 2800
-F 0 "C26" H 3865 2846 50  0000 L CNN
-F 1 "1nF" H 3865 2755 50  0000 L CNN
-F 2 "Capacitor_SMD:C_0402_1005Metric" H 3788 2650 50  0001 C CNN
-F 3 "~" H 3750 2800 50  0001 C CNN
-	1    3750 2800
-	-1   0    0    -1
+P 3050 2450
+F 0 "C26" H 3165 2496 50  0000 L CNN
+F 1 "1nF" H 3165 2405 50  0000 L CNN
+F 2 "Capacitor_SMD:C_0402_1005Metric" H 3088 2300 50  0001 C CNN
+F 3 "~" H 3050 2450 50  0001 C CNN
+	1    3050 2450
+	1    0    0    -1
 $EndComp
 $Comp
 L power:VDD #PWR063
 U 1 1 609C5138
-P 3400 2350
-F 0 "#PWR063" H 3400 2200 50  0001 C CNN
-F 1 "VDD" H 3415 2523 50  0000 C CNN
-F 2 "" H 3400 2350 50  0001 C CNN
-F 3 "" H 3400 2350 50  0001 C CNN
-	1    3400 2350
-	-1   0    0    -1
-$EndComp
-Wire Wire Line
-	3400 3300 3400 2450
+P 3400 2000
+F 0 "#PWR063" H 3400 1850 50  0001 C CNN
+F 1 "VDD" H 3415 2173 50  0000 C CNN
+F 2 "" H 3400 2000 50  0001 C CNN
+F 3 "" H 3400 2000 50  0001 C CNN
+	1    3400 2000
+	1    0    0    -1
+$EndComp
 Wire Wire Line
 	3300 3300 3400 3300
@@
 	7100 3600 6100 3600
 Wire Wire Line
-	4200 3450 3300 3450
+	4200 3450 4050 3450
 $Comp
 L Regular_Use:B4327 U6
@@
 	1    0    0    -1
 $EndComp
+NoConn ~ 5400 2850
+$Comp
+L Regular_Use:RF_Taper U12
+U 1 1 60A0B931
+P 5150 3100
+F 0 "U12" V 5134 3042 50  0000 R CNN
+F 1 "RF_Taper" V 5043 3042 50  0000 R CNN
+F 2 "ASSETS:KL_Taper" H 5050 3300 50  0001 C CNN
+F 3 "" H 5050 3300 50  0001 C CNN
+	1    5150 3100
+	0    -1   -1   0
+$EndComp
+Wire Wire Line
+	5150 3300 5150 3450
+Connection ~ 5150 3450
+Wire Wire Line
+	5150 3450 5050 3450
+$Comp
+L Regular_Use:RF_Taper U11
+U 1 1 60A0DC6F
+P 4050 3100
+F 0 "U11" V 4034 3042 50  0000 R CNN
+F 1 "RF_Taper" V 3943 3042 50  0000 R CNN
+F 2 "ASSETS:KL_Taper" H 3950 3300 50  0001 C CNN
+F 3 "" H 3950 3300 50  0001 C CNN
+	1    4050 3100
+	0    -1   -1   0
+$EndComp
+Wire Wire Line
+	4050 3300 4050 3450
+Connection ~ 4050 3450
+Wire Wire Line
+	4050 3450 3500 3450
+$Comp
+L Regular_Use:RF_Taper U10
+U 1 1 60A0FCC2
+P 3550 2850
+F 0 "U10" V 3534 2792 50  0000 R CNN
+F 1 "RF_Taper" V 3443 2792 50  0000 R CNN
+F 2 "ASSETS:KL_Taper" H 3450 3050 50  0001 C CNN
+F 3 "" H 3450 3050 50  0001 C CNN
+	1    3550 2850
+	0    -1   -1   0
+$EndComp
+Wire Wire Line
+	3400 2100 3400 3300
+Wire Wire Line
+	3550 3050 3500 3050
+Wire Wire Line
+	3500 3050 3500 3450
+Connection ~ 3500 3450
+Wire Wire Line
+	3500 3450 3300 3450
+$Comp
+L Regular_Use:RF_Taper U9
+U 1 1 60A16A72
+P 2250 2850
+F 0 "U9" V 2234 2792 50  0000 R CNN
+F 1 "RF_Taper" V 2143 2792 50  0000 R CNN
+F 2 "ASSETS:KL_Taper" H 2150 3050 50  0001 C CNN
+F 3 "" H 2150 3050 50  0001 C CNN
+	1    2250 2850
+	0    -1   -1   0
+$EndComp
+Wire Wire Line
+	2250 3050 2250 3600
+Connection ~ 2250 3600
+Wire Wire Line
+	2250 3600 2300 3600
 $EndSCHEMATC

Commit message: Add files via upload
Parts:
- removed U10: RF_Taper, ASSETS:KL_Taper, symbol Regular_Use:RF_Taper
- added U3: RF_Taper, ASSETS:KL_Taper, symbol Regular_Use:RF_Taper
Connections:
- net VDD: now also U3.1 (Tap)
Changed lines of the file:
@@
 Connection ~ 4050 3450
 Wire Wire Line
-	4050 3450 3500 3450
-$Comp
-L Regular_Use:RF_Taper U10
-U 1 1 60A0FCC2
-P 3550 2850
-F 0 "U10" V 3534 2792 50  0000 R CNN
-F 1 "RF_Taper" V 3443 2792 50  0000 R CNN
-F 2 "ASSETS:KL_Taper" H 3450 3050 50  0001 C CNN
-F 3 "" H 3450 3050 50  0001 C CNN
-	1    3550 2850
-	0    -1   -1   0
-$EndComp
-Wire Wire Line
-	3400 2100 3400 3300
-Wire Wire Line
-	3550 3050 3500 3050
-Wire Wire Line
-	3500 3050 3500 3450
-Connection ~ 3500 3450
-Wire Wire Line
-	3500 3450 3300 3450
+	3400 2100 3400 2400
 $Comp
 L Regular_Use:RF_Taper U9
@@
 Wire Wire Line
 	2250 3600 2300 3600
+$Comp
+L Regular_Use:RF_Taper U3
+U 1 1 60A8E179
+P 3650 2400
+F 0 "U3" V 3634 2342 50  0000 R CNN
+F 1 "RF_Taper" H 3850 2500 50  0000 R CNN
+F 2 "ASSETS:KL_Taper" H 3550 2600 50  0001 C CNN
+F 3 "" H 3550 2600 50  0001 C CNN
+	1    3650 2400
+	1    0    0    -1
+$EndComp
+Wire Wire Line
+	3450 2400 3400 2400
+Connection ~ 3400 2400
+Wire Wire Line
+	3400 2400 3400 3300
+Wire Wire Line
+	3300 3450 4050 3450
 $EndSCHEMATC

Commit message: Add files via upload
Connections:
- net VBAT is gone; now on an unnamed net: U7.6 (VBATT)
- net VDD renamed VCC_RF
Changed lines of the file:
@@
 Wire Wire Line
 	3300 3800 3500 3800
-Wire Wire Line
-	3400 2100 3400 2000
 Connection ~ 3400 2100
 Wire Wire Line
@@
 F 3 "~" H 3050 2450 50  0001 C CNN
 	1    3050 2450
-	1    0    0    -1
-$EndComp
-$Comp
-L power:VDD #PWR063
-U 1 1 609C5138
-P 3400 2000
-F 0 "#PWR063" H 3400 1850 50  0001 C CNN
-F 1 "VDD" H 3415 2173 50  0000 C CNN
-F 2 "" H 3400 2000 50  0001 C CNN
-F 3 "" H 3400 2000 50  0001 C CNN
-	1    3400 2000
 	1    0    0    -1
 $EndComp
@@
 	1    0    0    -1
 $EndComp
-$Comp
-L power:VDD #PWR068
-U 1 1 60A707E6
-P 6450 3750
-F 0 "#PWR068" H 6450 3600 50  0001 C CNN
-F 1 "VDD" H 6465 3923 50  0000 C CNN
-F 2 "" H 6450 3750 50  0001 C CNN
-F 3 "" H 6450 3750 50  0001 C CNN
-	1    6450 3750
-	0    -1   1    0
-$EndComp
 Wire Wire Line
 	8950 3400 8500 3400
@@
 Wire Wire Line
 	8500 3300 8950 3300
-Text GLabel 8650 3050 1    50   Input ~ 0
-VBAT
 Wire Wire Line
 	8650 3200 8650 3050
@@
 Wire Wire Line
 	3300 3450 4050 3450
+Wire Wire Line
+	8650 3050 8950 3050
+Wire Wire Line
+	8950 3050 8950 3300
+Connection ~ 8950 3300
+Text GLabel 6450 3750 0    50   Input ~ 0
+VCC_RF
+Text GLabel 3200 1900 0    50   Input ~ 0
+VCC_RF
+Wire Wire Line
+	3200 1900 3400 1900
+Wire Wire Line
+	3400 1900 3400 2100
 $EndSCHEMATC
