File: Hardware/Schematic/MCU.sch (KiCad schematic (older format))
At the start: 12 parts

Commit message: Add files via upload
Changed lines of the file:
@@
 $Descr A4 11693 8268
 encoding utf-8
-Sheet 2 4
-Title ""
-Date ""
-Rev ""
-Comp ""
+Sheet 2 5
+Title "ProRTK: All in one Real Time Kinematic device"
+Date "2021-05-12"
+Rev "1"
+Comp "Blackshield Engineering"
 Comment1 ""
 Comment2 ""
@@
 Wire Wire Line
 	2900 3650 2900 3450
+Text GLabel 8950 3550 2    50   Input ~ 0
+D+
+Text GLabel 8950 3650 2    50   Input ~ 0
+D-
+Text GLabel 9800 4000 2    50   Input ~ 0
+SDA_ALT
+Text GLabel 9800 3800 2    50   Input ~ 0
+SCL_ALT
+Text GLabel 9250 4700 0    50   Input ~ 0
+SDA_IMU
+Text GLabel 9250 4600 0    50   Input ~ 0
+SCL_IMU
+Text GLabel 9200 4500 0    50   Input ~ 0
+BOOT
+Text GLabel 9150 4300 0    50   Input ~ 0
+INT
+Text GLabel 9300 4100 0    50   Input ~ 0
+nRESET
+Text GLabel 8200 5100 2    50   Input ~ 0
+SDA
+Text GLabel 8200 4900 2    50   Input ~ 0
+SCL
+Text GLabel 8150 4700 2    50   Input ~ 0
+1PPS
+Text GLabel 8150 4500 2    50   Input ~ 0
+SYS_RSTN
+Text GLabel 8150 4400 2    50   Input ~ 0
+WAKE-UP
+Text GLabel 8150 4300 2    50   Input ~ 0
+RX_GNSS
+Text GLabel 8150 4200 2    50   Input ~ 0
+TX_GNSS
+Text GLabel 8550 4000 0    50   Input ~ 0
+SDA_GNSS
+Text GLabel 8550 4100 0    50   Input ~ 0
+SCL_GNSS
+Text GLabel 8200 3850 2    50   Input ~ 0
+LED3
+Text GLabel 8200 3750 2    50   Input ~ 0
+LED2
+Text GLabel 8200 3650 2    50   Input ~ 0
+LED1
+Text GLabel 8150 3300 2    50   Input ~ 0
+DAT0
+Text GLabel 8150 3400 2    50   Input ~ 0
+DAT1
+Text GLabel 8150 3200 2    50   Input ~ 0
+CLK
+Text GLabel 8150 3100 2    50   Input ~ 0
+CMD
+Text GLabel 8150 2900 2    50   Input ~ 0
+DAT2
+Text GLabel 8150 3000 2    50   Input ~ 0
+DAT3
 $EndSCHEMATC

Commit message: Add files via upload
Parts:
- added Y?: NX2012SA-32.768K-STD-MUB-1, ASSETS:NX2012SA32768KSTDMUB1, symbol Regular_Use:NX2012SA-32.768K-STD-MUB-1
- added Y?: NX2016SA-32M-EXS00A-CS06465, ASSETS:NX2016SA32MEXS00ACS06465, symbol Regular_Use:NX2016SA-32M-EXS00A-CS06465
Connections:
- net 1PPS: now also U?.26 (PB13)
- net BOOT: now also U?.15 (PA5)
- net CLK: now also U?.28 (PB15)
- net CMD: now also U?.16 (PA6)
- net D+: now also U?.32 (PA11)
- net D-: now also U?.33 (PA12)
- net DAT0: now also U?.40 (PB4)
- net DAT1: now also U?.29 (PA8)
- net DAT2: now also U?.30 (PA9)
- net DAT3: now also U?.41 (PB5)
- net GND: now also Y?.2 (GND_1), Y?.4 (GND_2)
- net INT: now also U?.14 (PA4)
- net LED1: now also U?.18 (PB0)
- net LED2: now also U?.19 (PB1)
- net LED3: now also U?.20 (PB2)
- net RX_GNSS: now also U?.38 (PA15)
- net SCL_ALT: now also U?.21 (PB10)
- net SCL_GNSS: now also U?.42 (PB6)
- net SDA_ALT: now also U?.46 (PB9)
- net SDA_GNSS: now also U?.43 (PB7)
- net SYS_RSTN: now also U?.31 (PA10)
- net TX_GNSS: now also U?.39 (PB3)
- net WAKE-UP: now also U?.17 (PA7)
- net X32_IN: now also Y?.1 (CRYSTAL_1)
- net X32_OUT: now also Y?.2 (CRYSTAL_2)
- net XOSC_IN: now also Y?.1 (CRYSTAL_1)
- net XOSC_OUT: now also Y?.3 (CRYSTAL_2)
- net nRESET: now also U?.10 (PA0)
- net EN: now reaches U?.11 (PA1)
- net ESP_RX: now reaches U?.12 (PA2)
- net EXP_TX: now reaches U?.13 (PA3)
- net SWDIO: now reaches U?.34 (PA13)
- net SWCLK: now reaches U?.37 (PA14)
- no-connect marks 0 -> 3
Changed lines of the file:
@@
 Wire Wire Line
 	2900 3650 2900 3450
-Text GLabel 8950 3550 2    50   Input ~ 0
+Text GLabel 6100 4150 2    50   Input ~ 0
+EXP_TX
+Text GLabel 6100 4050 2    50   Input ~ 0
+ESP_RX
+Text GLabel 6100 3950 2    50   Input ~ 0
+EN
+Text GLabel 3750 4850 0    50   Input ~ 0
+SDA_ALT
+Text GLabel 3750 4950 0    50   Input ~ 0
+SCL_ALT
+Text GLabel 3750 5150 0    50   Input ~ 0
+1PPS
+Text GLabel 6050 4850 2    50   Input ~ 0
+SYS_RSTN
+Text GLabel 6050 4550 2    50   Input ~ 0
+WAKE-UP
+Text GLabel 6050 5350 2    50   Input ~ 0
+RX_GNSS
+Text GLabel 3650 4250 0    50   Input ~ 0
+TX_GNSS
+Text GLabel 3750 4650 0    50   Input ~ 0
+SDA_GNSS
+Text GLabel 3750 4550 0    50   Input ~ 0
+SCL_GNSS
+Text GLabel 6050 4950 2    50   Input ~ 0
 D+
-Text GLabel 8950 3650 2    50   Input ~ 0
+Text GLabel 6050 5050 2    50   Input ~ 0
 D-
-Text GLabel 9800 4000 2    50   Input ~ 0
-SDA_ALT
-Text GLabel 9800 3800 2    50   Input ~ 0
-SCL_ALT
-Text GLabel 9250 4700 0    50   Input ~ 0
+Text GLabel 3750 4350 0    50   Input ~ 0
+DAT0
+Text GLabel 6050 4650 2    50   Input ~ 0
+DAT1
+Text GLabel 3650 5350 0    50   Input ~ 0
+CLK
+Text GLabel 6050 4450 2    50   Input ~ 0
+CMD
+Text GLabel 6050 4750 2    50   Input ~ 0
+DAT2
+Text GLabel 3750 4450 0    50   Input ~ 0
+DAT3
+Text GLabel 3250 4850 0    50   Input ~ 0
 SDA_IMU
-Text GLabel 9250 4600 0    50   Input ~ 0
+Text GLabel 3250 4950 0    50   Input ~ 0
 SCL_IMU
-Text GLabel 9200 4500 0    50   Input ~ 0
+Text GLabel 6100 4350 2    50   Input ~ 0
 BOOT
-Text GLabel 9150 4300 0    50   Input ~ 0
+Text GLabel 6100 4250 2    50   Input ~ 0
 INT
-Text GLabel 9300 4100 0    50   Input ~ 0
+Text GLabel 6100 3850 2    50   Input ~ 0
 nRESET
-Text GLabel 8200 5100 2    50   Input ~ 0
-SDA
-Text GLabel 8200 4900 2    50   Input ~ 0
-SCL
-Text GLabel 8150 4700 2    50   Input ~ 0
-1PPS
-Text GLabel 8150 4500 2    50   Input ~ 0
-SYS_RSTN
-Text GLabel 8150 4400 2    50   Input ~ 0
-WAKE-UP
-Text GLabel 8150 4300 2    50   Input ~ 0
-RX_GNSS
-Text GLabel 8150 4200 2    50   Input ~ 0
-TX_GNSS
-Text GLabel 8550 4000 0    50   Input ~ 0
-SDA_GNSS
-Text GLabel 8550 4100 0    50   Input ~ 0
-SCL_GNSS
-Text GLabel 8200 3850 2    50   Input ~ 0
+Text GLabel 3650 3950 0    50   Input ~ 0
+LED1
+Text GLabel 3650 4050 0    50   Input ~ 0
+LED2
+Text GLabel 3650 4150 0    50   Input ~ 0
 LED3
-Text GLabel 8200 3750 2    50   Input ~ 0
-LED2
-Text GLabel 8200 3650 2    50   Input ~ 0
-LED1
-Text GLabel 8150 3300 2    50   Input ~ 0
-DAT0
-Text GLabel 8150 3400 2    50   Input ~ 0
-DAT1
-Text GLabel 8150 3200 2    50   Input ~ 0
-CLK
-Text GLabel 8150 3100 2    50   Input ~ 0
-CMD
-Text GLabel 8150 2900 2    50   Input ~ 0
-DAT2
-Text GLabel 8150 3000 2    50   Input ~ 0
-DAT3
+$Comp
+L Regular_Use:NX2012SA-32.768K-STD-MUB-1 Y?
+U 1 1 60CC6D57
+P 8800 2550
+F 0 "Y?" H 9509 2546 50  0000 L CNN
+F 1 "NX2012SA-32.768K-STD-MUB-1" H 9509 2455 50  0000 L CNN
+F 2 "ASSETS:NX2012SA32768KSTDMUB1" H 9850 2650 50  0001 L CNN
+F 3 "https://www.mouser.de/datasheet/2/905/c_NX2012SA-STD-MUB-1_e-1317508.pdf" H 9850 2550 50  0001 L CNN
+F 4 "NDK 32.76kHz Crystal Unit +/-20ppm SMD 2-Pin 2.05 x 1.2 x 0.55mm" H 9850 2450 50  0001 L CNN "Description"
+F 5 "0.6" H 9850 2350 50  0001 L CNN "Height"
+F 6 "344-NX2012SA32768K1" H 9850 2250 50  0001 L CNN "Mouser Part Number"
+F 7 "https://www.mouser.co.uk/ProductDetail/NDK/NX2012SA-32768K-STD-MUB-1?qs=55YtniHzbhA%252B6%2Fl1MwFZaQ%3D%3D" H 9850 2150 50  0001 L CNN "Mouser Price/Stock"
+F 8 "NDK" H 9850 2050 50  0001 L CNN "Manufacturer_Name"
+F 9 "NX2012SA-32.768K-STD-MUB-1" H 9850 1950 50  0001 L CNN "Manufacturer_Part_Number"
+	1    8800 2550
+	1    0    0    -1
+$EndComp
+$Comp
+L Regular_Use:NX2016SA-32M-EXS00A-CS06465 Y?
+U 1 1 60CC7351
+P 8850 5200
+F 0 "Y?" H 9450 5465 50  0000 C CNN
+F 1 "NX2016SA-32M-EXS00A-CS06465" H 9450 5374 50  0000 C CNN
+F 2 "ASSETS:NX2016SA32MEXS00ACS06465" H 9900 5300 50  0001 L CNN
+F 3 "http://www.ndk.com/images/products/catalog/c_NX2016SA_e.pdf" H 9900 5200 50  0001 L CNN
+F 4 "CRYSTAL 32MHZ 10PF SMD" H 9900 5100 50  0001 L CNN "Description"
+F 5 "0.5" H 9900 5000 50  0001 L CNN "Height"
+F 6 "344-NX2016SA32S06465" H 9900 4900 50  0001 L CNN "Mouser Part Number"
+F 7 "https://www.mouser.co.uk/ProductDetail/NDK/NX2016SA-32M-EXS00A-CS06465?qs=w%2Fv1CP2dgqr82b0JjRnv4A%3D%3D" H 10300 4800 50  0001 L CNN "Mouser Price/Stock"
+F 8 "NDK" H 10300 4700 50  0001 L CNN "Manufacturer_Name"
+F 9 "NX2016SA-32M-EXS00A-CS06465" H 10300 4600 50  0001 L CNN "Manufacturer_Part_Number"
+	1    8850 5200
+	1    0    0    -1
+$EndComp
+Wire Wire Line
+	3650 4250 4200 4250
+Wire Wire Line
+	5500 5350 6050 5350
+Wire Wire Line
+	6100 4050 5500 4050
+Wire Wire Line
+	5500 4150 6100 4150
+Wire Wire Line
+	6050 4950 5500 4950
+Wire Wire Line
+	5500 5050 6050 5050
+Wire Wire Line
+	3750 4550 4200 4550
+Wire Wire Line
+	3750 4650 4200 4650
+Wire Wire Line
+	3750 4850 3850 4850
+Wire Wire Line
+	3750 4950 3850 4950
+Wire Wire Line
+	6100 3950 5500 3950
+Wire Wire Line
+	6050 4750 5500 4750
+Wire Wire Line
+	5500 4650 6050 4650
+Wire Wire Line
+	3650 5350 4200 5350
+Wire Wire Line
+	3750 4350 4200 4350
+Wire Wire Line
+	3750 4450 4200 4450
+Wire Wire Line
+	6050 4450 5500 4450
+Wire Wire Line
+	3350 4850 3350 4750
+Wire Wire Line
+	3350 4750 3850 4750
+Wire Wire Line
+	3850 4750 3850 4850
+Wire Wire Line
+	3250 4850 3350 4850
+Connection ~ 3850 4850
+Wire Wire Line
+	3850 4850 4200 4850
+Wire Wire Line
+	3250 4950 3350 4950
+Wire Wire Line
+	3350 4950 3350 5050
+Wire Wire Line
+	3350 5050 3850 5050
+Wire Wire Line
+	3850 5050 3850 4950
+Connection ~ 3850 4950
+Wire Wire Line
+	3850 4950 4200 4950
+Wire Wire Line
+	5500 5150 6050 5150
+Text GLabel 6050 5150 2    50   Input ~ 0
+SWDIO
+Wire Wire Line
+	5500 5250 6050 5250
+Text GLabel 6050 5250 2    50   Input ~ 0
+SWCLK
+Text GLabel 8550 5300 0    50   Input ~ 0
+XOSC_IN
+Text GLabel 10300 5200 2    50   Input ~ 0
+XOSC_OUT
+Wire Wire Line
+	10050 5200 10300 5200
+Wire Wire Line
+	8550 5300 8850 5300
+Wire Wire Line
+	8850 5200 8700 5200
+Wire Wire Line
+	8700 5200 8700 4850
+Wire Wire Line
+	8700 4850 8400 4850
+Wire Wire Line
+	8400 4850 8400 5000
+$Comp
+L power:GND #PWR?
+U 1 1 60D80852
+P 8400 5000
+F 0 "#PWR?" H 8400 4750 50  0001 C CNN
+F 1 "GND" H 8405 4827 50  0000 C CNN
+F 2 "" H 8400 5000 50  0001 C CNN
+F 3 "" H 8400 5000 50  0001 C CNN
+	1    8400 5000
+	1    0    0    -1
+$EndComp
+Wire Wire Line
+	10050 5300 10350 5300
+Wire Wire Line
+	10350 5300 10350 5450
+$Comp
+L power:GND #PWR?
+U 1 1 60D8104F
+P 10350 5450
+F 0 "#PWR?" H 10350 5200 50  0001 C CNN
+F 1 "GND" H 10355 5277 50  0000 C CNN
+F 2 "" H 10350 5450 50  0001 C CNN
+F 3 "" H 10350 5450 50  0001 C CNN
+	1    10350 5450
+	-1   0    0    -1
+$EndComp
+Text GLabel 8500 2550 0    50   Input ~ 0
+X32_IN
+Text GLabel 8500 2650 0    50   Input ~ 0
+X32_OUT
+Wire Wire Line
+	8500 2550 8800 2550
+Wire Wire Line
+	8500 2650 8800 2650
+Wire Wire Line
+	3650 3950 4200 3950
+Wire Wire Line
+	4200 4050 3650 4050
+Wire Wire Line
+	3650 4150 4200 4150
+Wire Wire Line
+	6100 3850 5500 3850
+Wire Wire Line
+	6100 4250 5500 4250
+Wire Wire Line
+	5500 4350 6100 4350
+Wire Wire Line
+	6050 4550 5500 4550
+Wire Wire Line
+	6050 4850 5500 4850
+Wire Wire Line
+	3750 5150 4200 5150
+NoConn ~ 4200 4750
+NoConn ~ 4200 5050
+NoConn ~ 4200 5250
 $EndSCHEMATC

Commit message: Add files via upload
Parts:
- removed C? (x6): C, symbol Device:C
- added C10, C14, C16: 0.1nF, Capacitor_SMD:C_0402_1005Metric, symbol Device:C
- added C11, C12: C, Capacitor_SMD:C_0402_1005Metric, symbol Device:C
- added C13, C15, C9: 1uF, Capacitor_SMD:C_0402_1005Metric, symbol Device:C
- C5: renamed from C?; value C -> 4.7uF; footprint (none) -> Capacitor_SMD:C_0402_1005Metric
- C6: renamed from C?; footprint (none) -> Capacitor_SMD:C_0402_1005Metric
- C7: renamed from C?; value C -> 1uF; footprint (none) -> Capacitor_SMD:C_0402_1005Metric
- C8: renamed from C?; value C -> 0.1nF; footprint (none) -> Capacitor_SMD:C_0402_1005Metric
- R9: renamed from R?; footprint (none) -> Resistor_SMD:R_0402_1005Metric
- gave numbers to parts that had none: 3
Connections:
- net +3V3: now also C10.1, C13.1, C14.1, C15.1, C16.1, C9.1
- net GND: now also C10.2, C11.1, C12.1, C13.2, C14.2, C15.2, C16.2, C9.2
- net X32_IN: now also C11.2
- net X32_OUT: now also C12.2
Other:
- moved on the sheet: C5, C6, C7, C8, R9, U1, Y1, Y2

Commit message: Add files via upload
Connections:
- net VBAT is gone; now on net +3V3: U1.1 (VBAT)
Changed lines of the file:
@@
 Wire Wire Line
 	3900 2400 3900 2150
-Text GLabel 3900 2150 0    50   Input ~ 0
-VBAT
 Wire Wire Line
 	4000 2400 4000 2250
@@
 Wire Wire Line
 	2400 3000 2100 3000
+Wire Wire Line
+	3900 2150 4000 2150
+Wire Wire Line
+	4000 2150 4000 2250
+Connection ~ 4000 2250
 $EndSCHEMATC
