File: Hardware/Schematic/ProRTK.kicad_pcb (KiCad board)
At the start: 2 copper layers, 141 parts, among them IC1 ST1S12GR, IC2 ESP32-C3, J1 USB_SMD_105450-0101, J2 Micro_SD_Card, J4 SMA_Angled, J5 SMA_Angled, Q1 BC817, Q2 BC817, Q3 BC817, U1 STM32F411CEUx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

Commit message: Add files via upload
Parts:
- removed U3: MC-146, Crystal:Crystal_SMD_SeikoEpson_MC146-4Pin_6.7x1.5mm
- added U10: RF_Taper, ASSETS:KL_Taper, F.Cu at (3.70, 127.2)
- added U11: RF_Taper, ASSETS:KL_Taper, F.Cu at (1.10, 127.3)
- added U12: RF_Taper, ASSETS:KL_Taper, F.Cu at (-0.10, 127.6)
- added U9: RF_Taper, ASSETS:KL_Taper, F.Cu at (21.2, 119.5)
- added Y5: NX2012SA-32.768K-STD-MUB-1, ASSETS:NX2012SA32768KSTDMUB1, F.Cu at (137.9, 85.5)
- C10, C13, C14, C15, C16, C5, C6, C7, C8, C9: moved to F.Cu
- J2: moved to B.Cu
- moved D6 118.8 mm to (156.1, 125.8), turned to 270 degrees
- moved IC1 118.3 mm to (150.0, 130.3), turned to 180 degrees
- moved C3 109.2 mm to (153.2, 131.3)
- moved R3 106.6 mm to (152.7, 132.9), turned to 270 degrees
- moved U7 106.2 mm to (148.0, 53.0)
- moved C1 105.6 mm to (153.8, 127.6), turned to 90 degrees
- moved R1 105.1 mm to (152.6, 127.6), turned to 90 degrees
- moved R2 103.9 mm to (148.0, 130.3), turned to 180 degrees
- moved R8 103.7 mm to (156.1, 128.3), turned to 270 degrees
- moved D2 103.1 mm to (148.5, 123.1), turned to 270 degrees
- moved D4 102.6 mm to (147.0, 116.3), turned to 270 degrees
- moved D1 101.7 mm to (141.5, 126.6), turned to 90 degrees
- moved C4 99.5 mm to (143.9, 127.8)
- moved J2 99.2 mm to (126.9, 129.9), turned to 180 degrees
- moved Q3 98.7 mm to (143.3, 113.0), turned to 270 degrees
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Connections:
- C17 pad 1: VDD -> +3V3
- C19 pad 1: VDD -> +3V3
- C20 pad 1: VDD -> +3V3
- U2 pad 28: VDD -> +3V3
- U2 pad 3: VDD -> +3V3
Routing:
- net ESP_RX: track 0.00 -> 71.1 mm, vias 0 -> 2
- net EN: track 1.61 -> 64.0 mm
- net VDD: track 2.71 -> 48.4 mm, vias 0 -> 2
- net GND: track 19.8 -> 61.9 mm, vias 13 -> 51
- net nRESET: track 0.00 -> 33.9 mm
- net LED1: track 0.00 -> 25.5 mm, vias 0 -> 2
- net SCL_ALT: track 0.00 -> 21.6 mm, vias 0 -> 2
- net +3V3: track 15.8 -> 36.8 mm, vias 5 -> 0
- net LED2: track 0.00 -> 20.6 mm
- net LED3: track 0.00 -> 15.1 mm
- net SDA_ALT: track 0.00 -> 11.6 mm
- net SPIWP: track 0.00 -> 10.6 mm, vias 0 -> 2
- net Net-(R16-Pad1): track 0.00 -> 10.2 mm
- net SPICSO: track 0.00 -> 9.53 mm
- net SPICLK: track 0.00 -> 8.50 mm, vias 0 -> 2
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Other:
- board outline added: 50 x 100 mm

Commit message: Add files via upload
Parts:
- added H1: MountingHole, MountingHole:MountingHole_3.2mm_M3_Pad_Via, F.Cu at (176.0, 66.0)
- added H2: MountingHole, MountingHole:MountingHole_3.2mm_M3_Pad_Via, F.Cu at (176.0, 104.0)
- added H3: MountingHole, MountingHole:MountingHole_3.2mm_M3_Pad_Via, F.Cu at (244.0, 104.0)
- added H4: MountingHole, MountingHole:MountingHole_3.2mm_M3_Pad_Via, F.Cu at (244.0, 66.0)
- added H5: MountingHole, MountingHole:MountingHole_3.2mm_M3_Pad_Via, F.Cu at (210.0, 85.0)
- CR2023: footprint Battery:BatteryHolder_Keystone_1058_1x2032 -> Battery:BatteryHolder_Keystone_3034_1x20mm
- J2: moved to F.Cu
- moved C10 353.5 mm to (-215.6, 87.9), turned to 90 degrees
- moved C5 352.8 mm to (-216.3, 86.3), turned to 0 degrees
- moved C9 352.5 mm to (-214.6, 87.9), turned to 90 degrees
- moved C14 346.7 mm to (-206.9, 90.2), turned to 180 degrees
- moved C13 345.7 mm to (-206.9, 89.2), turned to 180 degrees
- moved U1 344.3 mm to (-209.9, 84.5), turned to 270 degrees
- moved C16 340.5 mm to (-211.0, 79.2), turned to 90 degrees
- moved R9 338.5 mm to (-211.8, 76.1), turned to 270 degrees
- moved C15 337.7 mm to (-204.2, 83.8), turned to 0 degrees
- moved Y1 336.6 mm to (-209.2, 77.0), turned to 135 degrees
- moved C7 336.6 mm to (-205.1, 81.6), turned to 270 degrees
- moved C8 335.4 mm to (-204.0, 81.6), turned to 270 degrees
- moved Y2 333.5 mm to (-206.4, 76.9), turned to 90 degrees
- moved C11 332.3 mm to (-204.5, 77.8), turned to 180 degrees
- moved C12 330.6 mm to (-204.5, 76.0), turned to 180 degrees
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- renumbered SPI1 to SPIQ1
Routing:
- net ESP_RX: track 71.1 -> 0.00 mm, vias 2 -> 0
- net GND: track 61.9 -> 0.35 mm, vias 51 -> 3
- net EN: track 64.0 -> 4.55 mm
- net VDD: track 48.4 -> 0.00 mm, vias 2 -> 0
- net nRESET: track 33.9 -> 0.00 mm
- net LED1: track 25.5 -> 0.00 mm, vias 2 -> 0
- net LED2: track 20.6 -> 0.00 mm
- net SCL_ALT: track 21.6 -> 2.22 mm, vias 2 -> 0
- net +3V3: track 36.8 -> 18.2 mm, vias 0 -> 1
- net LED3: track 15.1 -> 0.00 mm
- net Net-(IC2-Pad21): track 2.30 -> 16.9 mm
- net Net-(IC2-Pad23): track 2.43 -> 16.6 mm
- net Net-(IC2-Pad24): track 2.63 -> 16.8 mm
- net Net-(IC2-Pad20): track 2.51 -> 16.6 mm
- net Net-(IC2-Pad22): track 2.22 -> 16.3 mm
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- added copper zone on F.Cu, net +3V3
- added copper zone on B.Cu, net GND
Other:
- board size 50 x 100 mm -> 76 x 46 mm

Commit message: Add files via upload
Parts:
- removed U10: RF_Taper, ASSETS:KL_Taper
- added U3: RF_Taper, ASSETS:KL_Taper, F.Cu at (186.0, 74.8)
- C1, C15, C3, C34, CR2023, IC1, L1, R1, R2, R3: moved to B.Cu
- moved DAT3 531.7 mm to (234.7, 95.1)
- moved DAT2 530.2 mm to (234.7, 96.2)
- moved CLK1 529.7 mm to (234.7, 91.8), turned to 180 degrees
- moved C30 528.4 mm to (205.7, 71.1), turned to 270 degrees
- moved CMD1 528.3 mm to (234.7, 94.0), turned to 180 degrees
- moved L3 525.8 mm to (204.7, 71.1), turned to 90 degrees
- moved 3.3V1 524.5 mm to (228.7, 76.7)
- moved C29 523.2 mm to (203.7, 71.1)
- moved SDA1 522.8 mm to (218.5, 92.8)
- moved BOOT1 518.9 mm to (219.4, 100.3)
- moved DAT1 511.2 mm to (234.7, 88.5)
- moved DAT0 508.8 mm to (234.7, 89.6), turned to 180 degrees
- moved VDD1 508.1 mm to (230.0, 72.5)
- moved D-1 503.3 mm to (226.0, 75.1)
- moved INT1 499.0 mm to (221.3, 93.6)
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Routing:
- net VDD: track 0.00 -> 65.1 mm, vias 0 -> 1
- net GND: track 0.35 -> 34.0 mm, vias 3 -> 20
- net +3V3: track 18.2 -> 42.7 mm, vias 1 -> 3
- net D+: track 0.00 -> 22.7 mm, vias 0 -> 2
- net D-: track 0.00 -> 19.5 mm
- net Net-(R16-Pad1): track 0.00 -> 10.4 mm, vias 0 -> 2
- net X32_OUT: track 0.00 -> 7.64 mm
- net X32_IN: track 0.00 -> 5.61 mm
- net NRST: track 0.00 -> 5.16 mm
- net Net-(C25-Pad2): track 0.00 -> 4.98 mm
- net ESP_RX: track 0.00 -> 4.51 mm
- net XOSC_IN: track 0.00 -> 4.41 mm
- net Net-(C27-Pad2): track 0.00 -> 4.37 mm
- net XOSC_OUT: track 0.00 -> 4.33 mm
- net Net-(C29-Pad1): track 0.00 -> 3.95 mm
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Other:
- copper layers 2 -> 4

Commit message: Add files via upload
Parts:
- removed CR2023: Conn_01x02, Battery:BatteryHolder_Keystone_3034_1x20mm
- added J3: Conn_01x01, ASSETS:Company_Logo1, F.Cu at (136.9, 99.5)
- C6: moved to B.Cu
- moved C6 121.9 mm to (163.5, 91.0)
- moved GND1 94.7 mm to (168.6, 92.7)
- moved SWDIO1 91.5 mm to (160.6, 102.6)
- moved SDA_ALT1 90.2 mm to (157.4, 108.7)
- moved SWCLK1 88.1 mm to (158.9, 102.6)
- moved 1PPS1 85.9 mm to (147.0, 90.7)
- moved GND2 85.1 mm to (174.2, 88.5)
- moved WAKE-UP1 80.0 mm to (148.0, 90.4)
- moved TX_GNSS1 79.1 mm to (145.8, 94.1)
- moved SCL_ALT1 77.7 mm to (156.5, 111.1)
- moved SYS_RSTN1 77.2 mm to (145.7, 84.8)
- moved DAT2 63.4 mm to (173.7, 113.5)
- moved CMD1 63.3 mm to (173.6, 110.4)
- moved CLK1 63.1 mm to (173.8, 108.5)
- moved DAT0 62.8 mm to (174.0, 105.8)
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Connections:
- C26 pad 1: VDD -> VCC_RF
- C28 pad 1: VDD -> VCC_RF
- J2 pad 4: VDD -> +3V3
- U1 pad 1: VBAT -> +3V3
- U3 pad 1: VDD -> VCC_RF
- U5 pad 2: VDD -> VCC_RF
- U7 pad 14: VDD -> VCC_RF
- U7 pad 6: VBAT -> Net-(C29-Pad1)
Routing:
- net GND: track 34.0 -> 104.6 mm, vias 20 -> 51
- net nRESET: track 1.86 -> 54.9 mm, vias 0 -> 3
- net SCL_GNSS: track 3.16 -> 47.8 mm, vias 0 -> 2
- net ESP_RX: track 4.51 -> 48.4 mm, vias 0 -> 2
- net CMD: track 0.00 -> 43.2 mm, vias 0 -> 2
- net SDA_GNSS: track 2.87 -> 44.5 mm, vias 0 -> 2
- net SYS_RSTN: track 0.00 -> 41.2 mm, vias 0 -> 2
- net BOOT: track 2.70 -> 43.7 mm, vias 0 -> 2
- net EN: track 4.55 -> 45.6 mm, vias 0 -> 4
- net SCL_ALT: track 3.23 -> 43.9 mm, vias 0 -> 4
- net EXP_TX: track 1.12 -> 40.8 mm, vias 0 -> 2
- net SDA_ALT: track 3.59 -> 38.8 mm, vias 0 -> 2
- net INT: track 2.48 -> 36.5 mm, vias 0 -> 2
- net DAT2: track 0.00 -> 32.8 mm, vias 0 -> 2
- net DAT3: track 0.00 -> 32.1 mm, vias 0 -> 2
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- added copper zone on In2.Cu, net +3V3
- added copper zone on In1.Cu, net GND
Other:
- rule trace_min: 0.2 -> 0.1
