File: Hardware/Schematic/ProRTK.sch (KiCad schematic (older format))
At the start: 37 parts

Commit message: Add files via upload
Parts:
- removed C? (x2): 1uF, symbol Device:C
- removed U?: AMS1117-3.3, Package_TO_SOT_SMD:SOT-223-3_TabPin2, symbol Regulator_Linear:AMS1117-3.3
- added 1PPS, RX_GNSS?, SCL_ALT, SCL_GNSS, SDA_ALT, SDA_GNSS, SYS_RSTN, TX_GNSS, WAKE-UP: TestPoint, symbol Connector:TestPoint
- added C? (x2): C, symbol Device:C
- added D?: SP0502BAJT, Package_TO_SOT_SMD:SOT-323_SC-70, symbol Power_Protection:SP0502BAJT
- added IC?: ST1S12GR, ASSETS:SOT95P280X110-5N, symbol Regular_Use:ST1S12GR
- added L?: L, symbol Device:L
- added R? (x3): R, symbol Device:R
Connections:
- net labels added: +3V3, 1PPS, RX_GNSS, SCL_ALT, SCL_GNSS, SCL_IMU, SDA_ALT, SDA_GNSS, SDA_IMU, SYS_RSTN, TX_GNSS, WAKE-UP
- net labels removed: SCL, SDA
- wire segments 92 -> 126
Other:
- moved on the sheet: 3.3V, CLK, CMD, CR2023, D+, D-, DAT0, DAT1, DAT2, DAT3, GND, VDD

Commit message: Add files via upload
Parts:
- added EN, ESP_RX, ESP_TX, MTCK, MTDI, MTDO, MTMS, SPI1, SPICLK, SPICSO, SPID, SPIHD, SPIWP: TestPoint, symbol Connector:TestPoint
Connections:
- new net EN: EN.1
- new net ESP_RX: ESP_RX.1
- new net EXP_TX: ESP_TX.1
- new net MTCK: MTCK.1
- new net MTDI: MTDI.1
- new net MTDO: MTDO.1
- new net MTMS: MTMS.1
- new net SPICLK: SPICLK.1
- new net SPICSO: SPICSO.1
- new net SPID: SPID.1
- new net SPIHD: SPIHD.1
- new net SPIQ: SPI1.1
- new net SPIWP: SPIWP.1
Changed lines of the file:
@@
 	9500 4550 10950 4550
 Wire Notes Line
-	11200 5700 9350 5700
-Wire Notes Line
-	9350 900  9350 5700
-Wire Notes Line
-	11200 500  11200 5700
+	11200 500  11200 6500
 $Sheet
-S 7000 3100 2300 3300
+S 7000 3150 2300 1950
 U 609C383C
 F0 "ESP32" 50
 F1 "ESP32.sch" 50
 $EndSheet
+Text GLabel 10600 5050 2    50   Input ~ 0
+SPIQ
+Text GLabel 10600 5200 2    50   Input ~ 0
+SPID
+Text GLabel 10600 5350 2    50   Input ~ 0
+SPICLK
+Text GLabel 10600 5500 2    50   Input ~ 0
+SPICSO
+Text GLabel 10600 5800 2    50   Input ~ 0
+SPIHD
+Text GLabel 10600 5650 2    50   Input ~ 0
+SPIWP
+Text GLabel 7200 5700 1    50   Input ~ 0
+EXP_TX
+Text GLabel 7350 5700 1    50   Input ~ 0
+ESP_RX
+Text GLabel 8750 5550 2    50   Input ~ 0
+EN
+Text GLabel 8750 5700 2    50   Input ~ 0
+MTMS
+Text GLabel 8750 5850 2    50   Input ~ 0
+MTDI
+Text GLabel 8750 6000 2    50   Input ~ 0
+MTCK
+Text GLabel 8750 6150 2    50   Input ~ 0
+MTDO
+$Comp
+L Connector:TestPoint SPID
+U 1 1 60B02F01
+P 10150 5200
+F 0 "SPID" V 10150 5400 50  0000 L CNN
+F 1 "TestPoint" V 10050 5150 50  0001 L CNN
+F 2 "" H 10350 5200 50  0001 C CNN
+F 3 "~" H 10350 5200 50  0001 C CNN
+	1    10150 5200
+	0    -1   -1   0
+$EndComp
+$Comp
+L Connector:TestPoint SPI1
+U 1 1 60B02F07
+P 10150 5050
+F 0 "SPI1" V 10150 5250 50  0000 L CNN
+F 1 "TestPoint" V 10050 5000 50  0001 L CNN
+F 2 "" H 10350 5050 50  0001 C CNN
+F 3 "~" H 10350 5050 50  0001 C CNN
+	1    10150 5050
+	0    -1   -1   0
+$EndComp
+$Comp
+L Connector:TestPoint SPICSO
+U 1 1 60B28901
+P 10150 5500
+F 0 "SPICSO" V 10150 5700 50  0000 L CNN
+F 1 "TestPoint" V 10050 5450 50  0001 L CNN
+F 2 "" H 10350 5500 50  0001 C CNN
+F 3 "~" H 10350 5500 50  0001 C CNN
+	1    10150 5500
+	0    -1   -1   0
+$EndComp
+$Comp
+L Connector:TestPoint SPICLK
+U 1 1 60B28907
+P 10150 5350
+F 0 "SPICLK" V 10150 5550 50  0000 L CNN
+F 1 "TestPoint" V 10050 5300 50  0001 L CNN
+F 2 "" H 10350 5350 50  0001 C CNN
+F 3 "~" H 10350 5350 50  0001 C CNN
+	1    10150 5350
+	0    -1   -1   0
+$EndComp
+$Comp
+L Connector:TestPoint SPIHD
+U 1 1 60B2E050
+P 10150 5800
+F 0 "SPIHD" V 10150 6000 50  0000 L CNN
+F 1 "TestPoint" V 10050 5750 50  0001 L CNN
+F 2 "" H 10350 5800 50  0001 C CNN
+F 3 "~" H 10350 5800 50  0001 C CNN
+	1    10150 5800
+	0    -1   -1   0
+$EndComp
+$Comp
+L Connector:TestPoint SPIWP
+U 1 1 60B2E056
+P 10150 5650
+F 0 "SPIWP" V 10150 5850 50  0000 L CNN
+F 1 "TestPoint" V 10050 5600 50  0001 L CNN
+F 2 "" H 10350 5650 50  0001 C CNN
+F 3 "~" H 10350 5650 50  0001 C CNN
+	1    10150 5650
+	0    -1   -1   0
+$EndComp
+Wire Wire Line
+	10150 5050 10600 5050
+Wire Wire Line
+	10600 5200 10150 5200
+Wire Wire Line
+	10150 5350 10600 5350
+Wire Wire Line
+	10600 5500 10150 5500
+Wire Wire Line
+	10150 5650 10600 5650
+Wire Wire Line
+	10150 5800 10600 5800
+Wire Notes Line
+	9500 5900 11100 5900
+Wire Notes Line
+	11100 5900 11100 4950
+Wire Notes Line
+	9500 4950 11100 4950
+Wire Notes Line
+	9500 4950 9500 5900
+Wire Notes Line
+	7000 5250 7000 6500
+Wire Notes Line
+	7000 6500 11200 6500
+Wire Notes Line
+	7000 5250 9350 5250
+Wire Notes Line
+	9350 5250 9350 500
+$Comp
+L Connector:TestPoint ESP_RX
+U 1 1 60B7FAB2
+P 7350 5900
+F 0 "ESP_RX" V 7350 6100 50  0000 L CNN
+F 1 "TestPoint" V 7250 5850 50  0001 L CNN
+F 2 "" H 7550 5900 50  0001 C CNN
+F 3 "~" H 7550 5900 50  0001 C CNN
+	1    7350 5900
+	-1   0    0    1
+$EndComp
+$Comp
+L Connector:TestPoint ESP_TX
+U 1 1 60B7FAB8
+P 7200 5900
+F 0 "ESP_TX" V 7200 6100 50  0000 L CNN
+F 1 "TestPoint" V 7100 5850 50  0001 L CNN
+F 2 "" H 7400 5900 50  0001 C CNN
+F 3 "~" H 7400 5900 50  0001 C CNN
+	1    7200 5900
+	-1   0    0    1
+$EndComp
+$Comp
+L Connector:TestPoint MTMS
+U 1 1 60B7FABE
+P 8050 5700
+F 0 "MTMS" V 8050 5900 50  0000 L CNN
+F 1 "TestPoint" V 7950 5650 50  0001 L CNN
+F 2 "" H 8250 5700 50  0001 C CNN
+F 3 "~" H 8250 5700 50  0001 C CNN
+	1    8050 5700
+	0    -1   -1   0
+$EndComp
+$Comp
+L Connector:TestPoint EN
+U 1 1 60B7FAC4
+P 8050 5550
+F 0 "EN" V 8050 5750 50  0000 L CNN
+F 1 "TestPoint" V 7950 5500 50  0001 L CNN
+F 2 "" H 8250 5550 50  0001 C CNN
+F 3 "~" H 8250 5550 50  0001 C CNN
+	1    8050 5550
+	0    -1   -1   0
+$EndComp
+$Comp
+L Connector:TestPoint MTCK
+U 1 1 60B7FACA
+P 8050 6000
+F 0 "MTCK" V 8050 6200 50  0000 L CNN
+F 1 "TestPoint" V 7950 5950 50  0001 L CNN
+F 2 "" H 8250 6000 50  0001 C CNN
+F 3 "~" H 8250 6000 50  0001 C CNN
+	1    8050 6000
+	0    -1   -1   0
+$EndComp
+$Comp
+L Connector:TestPoint MTDI
+U 1 1 60B7FAD0
+P 8050 5850
+F 0 "MTDI" V 8050 6050 50  0000 L CNN
+F 1 "TestPoint" V 7950 5800 50  0001 L CNN
+F 2 "" H 8250 5850 50  0001 C CNN
+F 3 "~" H 8250 5850 50  0001 C CNN
+	1    8050 5850
+	0    -1   -1   0
+$EndComp
+Wire Wire Line
+	7200 5900 7200 5700
+Wire Wire Line
+	7350 5700 7350 5900
+Wire Notes Line
+	7450 5300 7100 5300
+Wire Notes Line
+	7100 5300 7100 6400
+Wire Notes Line
+	7100 6400 7450 6400
+Wire Notes Line
+	7450 6400 7450 5300
+$Comp
+L Connector:TestPoint MTDO
+U 1 1 60BAB95C
+P 8050 6150
+F 0 "MTDO" V 8050 6350 50  0000 L CNN
+F 1 "TestPoint" V 7950 6100 50  0001 L CNN
+F 2 "" H 8250 6150 50  0001 C CNN
+F 3 "~" H 8250 6150 50  0001 C CNN
+	1    8050 6150
+	0    -1   -1   0
+$EndComp
+Wire Wire Line
+	8750 5550 8050 5550
+Wire Wire Line
+	8050 5700 8750 5700
+Wire Wire Line
+	8050 5850 8750 5850
+Wire Wire Line
+	8050 6000 8750 6000
+Wire Wire Line
+	8050 6150 8750 6150
+Wire Notes Line
+	9150 6300 9150 5400
+Wire Notes Line
+	7550 5400 7550 6300
+Wire Notes Line
+	7550 6300 9150 6300
+Wire Notes Line
+	7550 5400 9150 5400
+Wire Notes Line
+	2150 500  2150 1150
+Wire Notes Line
+	2150 1150 3550 1150
+Wire Notes Line
+	3550 1150 3550 500
+Wire Notes Line
+	3550 500  2150 500
 $EndSCHEMATC

Commit message: Add files via upload
Parts:
- added GND2, NRST1, SWCLK1, SWDIO1: TestPoint, ASSETS:testpoint_0.3mm, symbol Connector:TestPoint
- 1PPS1: renamed from 1PPS; footprint (none) -> ASSETS:testpoint_0.3mm
- 3.3V1: renamed from 3.3V; footprint (none) -> ASSETS:testpoint_0.3mm
- BOOT1: renamed from BOOT; footprint (none) -> ASSETS:testpoint_0.3mm
- C1, C2, C3, C4: renamed from C?; footprint (none) -> Capacitor_SMD:C_0402_1005Metric
- CLK1: renamed from CLK; footprint (none) -> ASSETS:testpoint_0.3mm
- CMD1: renamed from CMD; footprint (none) -> ASSETS:testpoint_0.3mm
- CR2023: footprint (none) -> Battery:BatteryHolder_Keystone_1058_1x2032
- D+1: renamed from D+; footprint (none) -> ASSETS:testpoint_0.3mm
- D-1: renamed from D-; footprint (none) -> ASSETS:testpoint_0.3mm
- D2, D3, D4, D5, D6: renamed from D?; footprint (none) -> LED_SMD:LED_0603_1608Metric
- DAT0, DAT1, DAT2, DAT3, SPI1: footprint (none) -> ASSETS:testpoint_0.3mm
- EN1: renamed from EN; footprint (none) -> ASSETS:testpoint_0.3mm
- ESP_RX1: renamed from ESP_RX; footprint (none) -> ASSETS:testpoint_0.3mm
- ESP_TX1: renamed from ESP_TX; footprint (none) -> ASSETS:testpoint_0.3mm
- GND1: renamed from GND; footprint (none) -> ASSETS:testpoint_0.3mm
- INT1: renamed from INT; footprint (none) -> ASSETS:testpoint_0.3mm
- J2: renamed from J?; footprint (none) -> Connector_Card:microSD_HC_Hirose_DM3D-SF
- L1: renamed from L?; footprint (none) -> Inductor_SMD:L_0402_1005Metric
- MTCK1: renamed from MTCK; footprint (none) -> ASSETS:testpoint_0.3mm
- MTDI1: renamed from MTDI; footprint (none) -> ASSETS:testpoint_0.3mm
- MTDO1: renamed from MTDO; footprint (none) -> ASSETS:testpoint_0.3mm
- MTMS1: renamed from MTMS; footprint (none) -> ASSETS:testpoint_0.3mm
- R1, R2, R3, R4, R5, R6, R7, R8: renamed from R?; footprint (none) -> Resistor_SMD:R_0402_1005Metric
- RX_GNSS1: renamed from RX_GNSS?; footprint (none) -> ASSETS:testpoint_0.3mm
- SCL1: renamed from SCL; footprint (none) -> ASSETS:testpoint_0.3mm
- SCL_ALT1: renamed from SCL_ALT; footprint (none) -> ASSETS:testpoint_0.3mm
- SCL_GNSS1: renamed from SCL_GNSS; footprint (none) -> ASSETS:testpoint_0.3mm
- SDA1: renamed from SDA; footprint (none) -> ASSETS:testpoint_0.3mm
- SDA_ALT1: renamed from SDA_ALT; footprint (none) -> ASSETS:testpoint_0.3mm
- SDA_GNSS1: renamed from SDA_GNSS; footprint (none) -> ASSETS:testpoint_0.3mm
- SPICLK1: renamed from SPICLK; footprint (none) -> ASSETS:testpoint_0.3mm
- SPICSO1: renamed from SPICSO; footprint (none) -> ASSETS:testpoint_0.3mm
- SPID1: renamed from SPID; footprint (none) -> ASSETS:testpoint_0.3mm
- SPIHD1: renamed from SPIHD; footprint (none) -> ASSETS:testpoint_0.3mm
- SPIWP1: renamed from SPIWP; footprint (none) -> ASSETS:testpoint_0.3mm
- SYS_RSTN1: renamed from SYS_RSTN; footprint (none) -> ASSETS:testpoint_0.3mm
- TX_GNSS1: renamed from TX_GNSS; footprint (none) -> ASSETS:testpoint_0.3mm
- VDD1: renamed from VDD; footprint (none) -> ASSETS:testpoint_0.3mm
- WAKE-UP1: renamed from WAKE-UP; footprint (none) -> ASSETS:testpoint_0.3mm
- nRESET1: renamed from nRESET; footprint (none) -> ASSETS:testpoint_0.3mm
- gave numbers to parts that had none: 6
Connections:
- net GND: now also GND2.1
- net LED1: no longer Q2.1 (B), Q3.1 (B)
- new net LED2: Q2.1 (B)
- new net LED3: Q3.1 (B)
- new net NRST: NRST1.1
- new net SWCLK: SWCLK1.1
- new net SWDIO: SWDIO1.1
- no-connect marks 12 -> 16
Other:
- moved on the sheet: CR2023, EN1, MTCK1, MTDI1, MTDO1, MTMS1

Commit message: Add files via upload
Parts:
- added H1, H2, H3, H4, H5: MountingHole, MountingHole:MountingHole_3.2mm_M3_Pad_Via, symbol Mechanical:MountingHole
- CR2023: footprint Battery:BatteryHolder_Keystone_1058_1x2032 -> Battery:BatteryHolder_Keystone_3034_1x20mm
- renumbered SPI1 to SPIQ1
Changed lines of the file:
@@
 F 0 "CR2023" V 1200 1000 50  0000 R CNN
 F 1 "Conn_01x02" V 1050 1000 50  0000 R CNN
-F 2 "Battery:BatteryHolder_Keystone_1058_1x2032" H 900 950 50  0001 C CNN
+F 2 "Battery:BatteryHolder_Keystone_3034_1x20mm" H 900 950 50  0001 C CNN
 F 3 "~" H 900 950 50  0001 C CNN
 	1    900  950
@@
 $EndComp
 $Comp
-L Connector:TestPoint SPI1
+L Connector:TestPoint SPIQ1
 U 1 1 60B02F07
 P 10150 5050
-F 0 "SPI1" V 10150 5250 50  0000 L CNN
+F 0 "SPIQ1" V 10150 5250 50  0000 L CNN
 F 1 "TestPoint" V 10050 5000 50  0001 L CNN
 F 2 "ASSETS:testpoint_0.3mm" H 10350 5050 50  0001 C CNN
@@
 F1 "IMU.sch" 50
 $EndSheet
+$Comp
+L Mechanical:MountingHole H1
+U 1 1 60A47F18
+P 2300 650
+F 0 "H1" H 2400 696 50  0000 L CNN
+F 1 "MountingHole" H 2400 605 50  0000 L CNN
+F 2 "MountingHole:MountingHole_3.2mm_M3_Pad_Via" H 2300 650 50  0001 C CNN
+F 3 "~" H 2300 650 50  0001 C CNN
+	1    2300 650
+	1    0    0    -1
+$EndComp
+$Comp
+L Mechanical:MountingHole H4
+U 1 1 60A58EC5
+P 3400 650
+F 0 "H4" V 3446 750 50  0000 L CNN
+F 1 "MountingHole" V 3355 750 50  0000 L CNN
+F 2 "MountingHole:MountingHole_3.2mm_M3_Pad_Via" H 3400 650 50  0001 C CNN
+F 3 "~" H 3400 650 50  0001 C CNN
+	1    3400 650
+	0    -1   1    0
+$EndComp
+$Comp
+L Mechanical:MountingHole H3
+U 1 1 60A8D98E
+P 2900 850
+F 0 "H3" V 2946 950 50  0000 L CNN
+F 1 "MountingHole" V 2855 950 50  0000 L CNN
+F 2 "MountingHole:MountingHole_3.2mm_M3_Pad_Via" H 2900 850 50  0001 C CNN
+F 3 "~" H 2900 850 50  0001 C CNN
+	1    2900 850
+	0    -1   1    0
+$EndComp
+$Comp
+L Mechanical:MountingHole H5
+U 1 1 60A8DCE3
+P 3450 1050
+F 0 "H5" V 3496 1150 50  0000 L CNN
+F 1 "MountingHole" V 3405 1150 50  0000 L CNN
+F 2 "MountingHole:MountingHole_3.2mm_M3_Pad_Via" H 3450 1050 50  0001 C CNN
+F 3 "~" H 3450 1050 50  0001 C CNN
+	1    3450 1050
+	0    -1   1    0
+$EndComp
+$Comp
+L Mechanical:MountingHole H2
+U 1 1 60A8E0EF
+P 2300 1050
+F 0 "H2" V 2346 1150 50  0000 L CNN
+F 1 "MountingHole" V 2255 1150 50  0000 L CNN
+F 2 "MountingHole:MountingHole_3.2mm_M3_Pad_Via" H 2300 1050 50  0001 C CNN
+F 3 "~" H 2300 1050 50  0001 C CNN
+	1    2300 1050
+	0    1    -1   0
+$EndComp
 $EndSCHEMATC

Commit message: Add files via upload
Parts:
- removed CR2023: Conn_01x02, Battery:BatteryHolder_Keystone_3034_1x20mm, symbol Connector_Generic:Conn_01x02
- added J3: Conn_01x01, ASSETS:Company_Logo1, symbol Connector_Generic:Conn_01x01
Connections:
- net +3V3: now also J2.4 (VDD)
- net VDD: no longer J2.4 (VDD)
- no-connect marks 16 -> 17
Changed lines of the file:
@@
 	-1   0    0    -1
-$EndComp
-$Comp
-L power:VDD #PWR010
-U 1 1 60C28FCD
-P 3250 6850
-F 0 "#PWR010" H 3250 6700 50  0001 C CNN
-F 1 "VDD" H 3265 7023 50  0000 C CNN
-F 2 "" H 3250 6850 50  0001 C CNN
-F 3 "" H 3250 6850 50  0001 C CNN
-	1    3250 6850
-	1    0    0    -1
 $EndComp
 Text GLabel 2850 7400 2    50   Input ~ 0
@@
 Text GLabel 2850 6900 2    50   Input ~ 0
 CMD
-Wire Wire Line
-	3250 6850 3250 7000
 Wire Wire Line
 	2650 7000 3250 7000
@@
 Wire Notes Line
 	500  6150 3550 6150
-$Comp
-L Connector_Generic:Conn_01x02 CR2023
-U 1 1 60BC0B64
-P 900 950
-F 0 "CR2023" V 1200 1000 50  0000 R CNN
-F 1 "Conn_01x02" V 1050 1000 50  0000 R CNN
-F 2 "Battery:BatteryHolder_Keystone_3034_1x20mm" H 900 950 50  0001 C CNN
-F 3 "~" H 900 950 50  0001 C CNN
-	1    900  950
-	-1   0    0    1
-$EndComp
-Wire Wire Line
-	1100 950  1700 950
-Text GLabel 1800 950  2    50   Input ~ 0
-VBAT
-Wire Wire Line
-	1100 850  1200 850
-$Comp
-L power:GND #PWR03
-U 1 1 60BC8A28
-P 1300 800
-F 0 "#PWR03" H 1300 550 50  0001 C CNN
-F 1 "GND" H 1305 627 50  0000 C CNN
-F 2 "" H 1300 800 50  0001 C CNN
-F 3 "" H 1300 800 50  0001 C CNN
-	1    1300 800
-	0    -1   -1   0
-$EndComp
 Wire Notes Line
 	500  3500 2550 3500
@@
 Wire Notes Line
 	500  1150 500  500
-Wire Wire Line
-	1200 800  1200 850
-Wire Wire Line
-	1200 800  1300 800
 Wire Notes Line
 	2100 1150 2100 500
@@
 	2450 5700 2450 5800
 NoConn ~ 2200 5650
-$Comp
-L power:PWR_FLAG #FLG0103
-U 1 1 60AC62EF
-P 1700 750
-F 0 "#FLG0103" H 1700 825 50  0001 C CNN
-F 1 "PWR_FLAG" H 1700 923 50  0000 C CNN
-F 2 "" H 1700 750 50  0001 C CNN
-F 3 "~" H 1700 750 50  0001 C CNN
-	1    1700 750
-	1    0    0    -1
-$EndComp
-Wire Wire Line
-	1700 750  1700 950
-Connection ~ 1700 950
-Wire Wire Line
-	1700 950  1800 950
 NoConn ~ 800  4850
 NoConn ~ 800  5550
@@
 	0    1    -1   0
 $EndComp
+$Comp
+L power:+3V3 #PWR03
+U 1 1 60AAC486
+P 3250 6800
+F 0 "#PWR03" H 3250 6650 50  0001 C CNN
+F 1 "+3V3" H 3265 6973 50  0000 C CNN
+F 2 "" H 3250 6800 50  0001 C CNN
+F 3 "" H 3250 6800 50  0001 C CNN
+	1    3250 6800
+	1    0    0    -1
+$EndComp
+Wire Wire Line
+	3250 6800 3250 7000
+$Comp
+L Connector_Generic:Conn_01x01 J3
+U 1 1 60B08E3E
+P 1200 850
+F 0 "J3" H 1280 846 50  0000 L CNN
+F 1 "Conn_01x01" H 1280 801 50  0001 L CNN
+F 2 "ASSETS:Company_Logo1" H 1200 850 50  0001 C CNN
+F 3 "~" H 1200 850 50  0001 C CNN
+	1    1200 850
+	1    0    0    -1
+$EndComp
+NoConn ~ 1000 850
 $EndSCHEMATC
